File: kicad/test.sch (KiCad schematic (older format))
At the start: 18 parts

Commit message: #finished schematic
Parts:
- added P?: STATO a vite, symbol CONN_01X05
- added R4, R5, R? (x6): 330, symbol R
- added R? (x4): 47k, symbol R
- added SW? (x4): SW_PCB, symbol SW_PCB
- added U2: 74LS244, symbol 74LS244
- gave numbers to parts that had none: 17
Connections:
- net ACK: now also D8.2 (A), P?.1 (P1), R?.2, U2.18 (O0a); no longer D10.2 (A)
- net BUSY: now also D9.2 (A), P?.2 (P2), R?.2, U2.16 (O1a); no longer D11.2 (A)
- net ERROR: now also P?.5 (P5), U2.11 (I0b), U2.9 (O0b)
- net GND: now also R4.2, R?.2, R?.2, R?.2, SW?.1, SW?.1, SW?.1, SW?.1, SW?.~, SW?.~, SW?.~, SW?.~, U2.1 (OEa), U2.10 (GND), U2.19 (OEb)
- net PAPEROUT: now also D10.2 (A), P?.3 (P3), R?.2, U2.14 (O2a); no longer D9.2 (A)
- net SELECT: now also D11.2 (A), P?.4 (P4), R5.2, U2.12 (O3a); no longer D8.2 (A)
- net VCC: now also R?.1, R?.1, R?.1, R?.1, U2.20 (VCC)
- net at D8.1 (K): now also R?.1
- net at D9.1 (K): now also R?.1
- net at D10.1 (K): now also R?.1
- net at D11.1 (K): now also R4.1
- new net: R?.1, R?.2, SW?.2, SW?.~, U2.2 (I0a)
- new net: R?.1, R?.2, SW?.2, SW?.~, U2.4 (I1a)
- new net: R?.1, R?.2, SW?.2, SW?.~, U2.6 (I2a)
- new net: R5.1, R?.2, SW?.2, SW?.~, U2.8 (I3a)
- no-connect marks 11 -> 17
Other:
- moved on the sheet: D0, D1, D10, D11, D2, D3, D4, D5, D6, D7, D8, D9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

Commit message: #schematic pdf
Parts:
- gave numbers to parts that had none: 15
Changed lines of the file:
@@
 Sheet 1 1
 Title ""
-Date ""
-Rev ""
-Comp ""
+Date "2016-10-14"
+Rev "A"
+Comp "ISIS Newton di Varese"
 Comment1 ""
 Comment2 ""
@@
 ERROR
 $Comp
-L R R?
+L R R1
 U 1 1 58011E4D
 P 7000 2700
@@
 $EndComp
 $Comp
-L R R?
+L R R2
 U 1 1 58011EA6
 P 7350 2700
@@
 $EndComp
 $Comp
-L R R?
+L R R3
 U 1 1 58011EFF
 P 7700 2700
@@
 	5200 2400 5250 2400
 $Comp
-L SW_PCB SW?
+L SW_PCB SW1
 U 1 1 5801A7D7
 P 3500 2350
@@
 $EndComp
 $Comp
-L SW_PCB SW?
+L SW_PCB SW2
 U 1 1 5801A85A
 P 3900 2350
@@
 $EndComp
 $Comp
-L SW_PCB SW?
+L SW_PCB SW3
 U 1 1 5801A8C1
 P 4300 2350
@@
 $EndComp
 $Comp
-L SW_PCB SW?
+L SW_PCB SW4
 U 1 1 5801A92D
 P 4700 2350
@@
 	4800 2700 4800 2650
 $Comp
-L CONN_01X05 P?
+L CONN_01X05 JP3
 U 1 1 5801B871
 P 1550 1700
@@
 	1750 1900 5250 1900
 $Comp
-L R R?
+L R R6
 U 1 1 5801D05F
 P 2600 1600
@@
 	2450 1800 1750 1800
 $Comp
-L R R?
+L R R7
 U 1 1 5801D805
 P 2600 1400
@@
 $EndComp
 $Comp
-L R R?
+L R R8
 U 1 1 5801D876
 P 2600 1200
@@
 	3000 1200 3000 1500
 $Comp
-L R R?
+L R R9
 U 1 1 5801E7F4
 P 4750 1250
@@
 $EndComp
 $Comp
-L R R?
+L R R10
 U 1 1 5801EBF4
 P 4350 1250
@@
 $EndComp
 $Comp
-L R R?
+L R R11
 U 1 1 5801EC76
 P 3950 1250
@@
 $EndComp
 $Comp
-L R R?
+L R R12
 U 1 1 5801ED03
 P 3550 1250
